File: Schematic/proximity_sensor.sch (EAGLE design)
At the start: 4 parts, among them IC1 7805DT, U1 ATMEGA328P_PDIP

Commit message: Schematic Update
Parts:
- added C3: 1u, rcl:C-EU025-024X044
- added IC2: 74AC11032D, 74ac-logic:74AC11032D
- added J1: AVR_SPI_PRG_6PTH, SparkFun-Connectors:AVR_SPI_PRG_6PTH
- added JP2: (no value), SparkFun-Connectors:ARDUINO_SERIAL_PROGRAMPTH
- added LED1, LED2, LED3: (no value), led:LED3MM
- added R1: (no value), rcl:R-US_0414/5V
- added U$1, U$2, U$5: MMDT3904, SparkFun-DiscreteSemi:TRANSISTOR_NPN2UPMMDT3904
Connections:
- new net CTS: JP2.CTS
- new net DTR: C3.2, JP2.DTR
- new net MISO: J1.1, U1.PB4(MISO)
- new net MOSI: J1.4, U1.PB3(MOSI/OC2)
- new net N$1: IC2A.O, U$1G$1.B
- new net N$2: IC2B.O, U$1G$2.B
- new net N$3: IC2C.O, U$2G$1.B
- new net N$5: LED1.C, U$1G$1.C
- new net N$8: LED2.C, U$1G$2.C
- new net N$9: LED3.C, U$2G$1.C
- new net RESET: C3.1, J1.5, R1.1, U1.PC6(/RESET)
- new net RX: JP2.TXO, U1.PD0(RXD)
- new net SCK: J1.3, U1.PB5(SCK)
- new net TX: JP2.RXI, U1.PD1(TXD)
- new net VCC: JP2.VCC
- net +5V: now also J1.2, LED1.A, LED2.A, LED3.A, R1.2
- net GND: now also J1.6, JP2.GND, U$1G$1.E, U$1G$2.E, U$2G$1.E
Other:
- note added: "3 LED Array"
- moved on the sheet: U1

Commit message: Schematic update and meeting notes
Parts:
- removed U$5: MMDT3904, SparkFun-DiscreteSemi:TRANSISTOR_NPN2UPMMDT3904
- added IC3: 74HC08D, 74xx-eu:74HC08D
- added LED4, LED5, LED6: (no value), SparkFun-LED:LED-3MM-NO_SILK
- added Q1, Q2: FDS6890A, transistor-power:FDS6890A
- added U$3: SV74LV4052APWR2, SparkFun-AnalogIC:SV74LV4052APWR2
Connections:
- new net N$10: Q2B.S
- new net N$11: IC3A.O, Q1A.G
- new net N$12: IC3B.O, Q1B.G
- new net N$13: IC3C.O, Q2A.G
- new net N$4: LED5.A, Q1B.S
- new net N$6: LED4.A, Q1A.S
- new net N$7: LED6.A, Q2A.S
- net +5V: now also Q1A.D, Q1B.D, Q2A.D
- net GND: now also LED4.C, LED5.C, LED6.C
Other:
- moved on the sheet: IC2A, IC2B, IC2C, IC2D, LED1, LED2, LED3, U$1G$1, U$1G$2, U$2G$1, U$2G$2
