File: Schematic/mainboard/mainboard.sch (EAGLE design)
At the start: 15 parts, among them IC1 7805DT, IC2 74AC11032D, J1 AVR_SPI_PRG_6PTH, U1 ATMEGA328P_PDIP

Commit message: Breadboard Prototype
Parts:
- removed IC2: 74AC11032D, 74ac-logic:74AC11032D
- removed LED1, LED2, LED3: (no value), led:LED3MM
- removed U$1, U$2, U$5: MMDT3904, SparkFun-DiscreteSemi:TRANSISTOR_NPN2UPMMDT3904
- added JP1, JP3, JP4: (no value), SparkFun-Connectors:M04JST
- added U$3: SV74LV4052APWR2, SparkFun-AnalogIC:SV74LV4052APWR2
Connections:
- removed net N$1: IC2A.O, U$1G$1.B
- removed net N$2: IC2B.O, U$1G$2.B
- removed net N$3: IC2C.O, U$2G$1.B
- removed net N$5: LED1.C, U$1G$1.C
- removed net N$8: LED2.C, U$1G$2.C
- removed net N$9: LED3.C, U$2G$1.C
- net +5V: no longer LED1.A, LED2.A, LED3.A
- net GND: no longer U$1G$1.E, U$1G$2.E, U$2G$1.E
Other:
- note removed: "3 LED Array"
Changed lines of the file:
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@@
 <?xml version="1.0" encoding="utf-8"?>
 <!DOCTYPE eagle SYSTEM "eagle.dtd">
-<eagle version="6.3">
+<eagle version="7.1.0">
 <drawing>
 <settings>
@@
 <setting verticaltext="up"/>
 </settings>
-<grid distance="0.05" unitdist="inch" unit="inch" style="lines" multiple="2" display="yes" altdistance="0.01" altunitdist="inch" altunit="inch"/>
+<grid distance="0.1" unitdist="inch" unit="inch" style="lines" multiple="1" display="no" altdistance="0.01" altunitdist="inch" altunit="inch"/>
 <layers>
 <layer number="1" name="Top" color="4" fill="1" visible="no" active="no"/>
@@
 <part name="MOTORCYCLEBATTERY" library="supply2" deviceset="+12V" device=""/>
 <part name="U1" library="SparkFun-DigitalIC" deviceset="ATMEGA328P_PDIP" device=""/>
-<part name="U$1" library="SparkFun-DiscreteSemi" deviceset="TRANSISTOR_NPN2UP" device="MMDT3904" value="MMDT3904"/>
 <part name="J1" library="SparkFun-Connectors" deviceset="AVR_SPI_PRG_6" device="PTH"/>
 <part name="JP2" library="SparkFun-Connectors" deviceset="ARDUINO_SERIAL_PROGRAM" device="PTH"/>
-<part name="U$2" library="SparkFun-DiscreteSemi" deviceset="TRANSISTOR_NPN2UP" device="MMDT3904" value="MMDT3904"/>
-<part name="U$5" library="SparkFun-DiscreteSemi" deviceset="TRANSISTOR_NPN2UP" device="MMDT3904" value="MMDT3904"/>
-<part name="IC2" library="74ac-logic" deviceset="74AC11032" device="D"/>
 <part name="R1" library="rcl" deviceset="R-US_" device="0414/5V"/>
 <part name="C3" library="rcl" deviceset="C-EU" device="025-024X044" value="1u"/>
 <part name="GND2" library="supply1" deviceset="GND" device=""/>
-<part name="GND3" library="supply1" deviceset="GND" device=""/>
-<part name="LED1" library="led" deviceset="LED" device="3MM"/>
-<part name="LED2" library="led" deviceset="LED" device="3MM"/>
-<part name="LED3" library="led" deviceset="LED" device="3MM"/>
+<part name="U$3" library="SparkFun-AnalogIC" deviceset="SV74LV4052APWR" device="2"/>
+<part name="JP1" library="SparkFun-Connectors" deviceset="M04" device="JST"/>
+<part name="JP3" library="SparkFun-Connectors" deviceset="M04" device="JST"/>
+<part name="JP4" library="SparkFun-Connectors" deviceset="M04" device="JST"/>
 </parts>
 <sheets>
@@
 <wire x1="15.24" y1="236.22" x2="15.24" y2="266.7" width="0.1524" layer="97"/>
 <text x="16.51" y="267.97" size="1.778" layer="97">12V to 5V Linear Power Supply</text>
-<wire x1="15.24" y1="19.05" x2="137.16" y2="19.05" width="0.1524" layer="97"/>
-<wire x1="137.16" y1="19.05" x2="137.16" y2="77.47" width="0.1524" layer="97"/>
-<wire x1="137.16" y1="77.47" x2="15.24" y2="77.47" width="0.1524" layer="97"/>
-<wire x1="15.24" y1="77.47" x2="15.24" y2="19.05" width="0.1524" layer="97"/>
-<text x="16.51" y="78.74" size="1.778" layer="97">3 LED Array</text>
 </plain>
 <instances>
@@
 <instance part="MOTORCYCLEBATTERY" gate="+12V" x="10.16" y="259.08"/>
 <instance part="U1" gate="G$1" x="99.06" y="205.74"/>
-<instance part="U$1" gate="G$1" x="40.64" y="39.37"/>
-<instance part="U$1" gate="G$2" x="66.04" y="39.37"/>
 <instance part="J1" gate="G$1" x="35.56" y="175.26"/>
 <instance part="JP2" gate="G$1" x="38.1" y="203.2"/>
-<instance part="U$2" gate="G$1" x="91.44" y="39.37"/>
-<instance part="U$2" gate="G$2" x="116.84" y="39.37"/>
-<instance part="U$5" gate="G$1" x="375.92" y="144.78"/>
-<instance part="IC2" gate="A" x="33.02" y="62.23" rot="R270"/>
-<instance part="IC2" gate="B" x="58.42" y="62.23" rot="R270"/>
-<instance part="IC2" gate="C" x="83.82" y="62.23" rot="R270"/>
-<instance part="IC2" gate="D" x="109.22" y="62.23" rot="R270"/>
 <instance part="R1" gate="G$1" x="66.04" y="246.38" rot="R90"/>
 <instance part="C3" gate="G$1" x="55.88" y="231.14" rot="R270"/>
 <instance part="GND2" gate="1" x="50.8" y="160.02"/>
-<instance part="GND3" gate="1" x="81.28" y="22.86"/>
-<instance part="LED1" gate="G$1" x="43.18" y="54.61"/>
-<instance part="LED2" gate="G$1" x="68.58" y="54.61"/>
-<instance part="LED3" gate="G$1" x="93.98" y="54.61"/>
+<instance part="U$3" gate="G$1" x="187.96" y="203.2"/>
+<instance part="JP1" gate="G$1" x="226.06" y="226.06"/>
+<instance part="JP3" gate="G$1" x="226.06" y="205.74"/>
+<instance part="JP4" gate="G$1" x="86.36" y="256.54"/>
 </instances>
 <busses>
@@
 <pinref part="GND2" gate="1" pin="GND"/>
 </segment>
-<segment>
-<pinref part="U$1" gate="G$1" pin="E"/>
-<wire x1="43.18" y1="34.29" x2="43.18" y2="29.21" width="0.1524" layer="91"/>
-<wire x1="43.18" y1="29.21" x2="68.58" y2="29.21" width="0.1524" layer="91"/>
-<wire x1="68.58" y1="29.21" x2="81.28" y2="29.21" width="0.1524" layer="91"/>
-<wire x1="81.28" y1="29.21" x2="93.98" y2="29.21" width="0.1524" layer="91"/>
-<pinref part="U$2" gate="G$1" pin="E"/>
-<wire x1="93.98" y1="29.21" x2="93.98" y2="34.29" width="0.1524" layer="91"/>
-<pinref part="U$1" gate="G$2" pin="E"/>
-<wire x1="68.58" y1="34.29" x2="68.58" y2="29.21" width="0.1524" layer="91"/>
-<junction x="68.58" y="29.21"/>
-<wire x1="81.28" y1="29.21" x2="81.28" y2="25.4" width="0.1524" layer="91"/>
-<junction x="81.28" y="29.21"/>
-<pinref part="GND3" gate="1" pin="GND"/>
-<wire x1="81.28" y1="25.4" x2="81.28" y2="24.13" width="0.1524" layer="91"/>
-<junction x="81.28" y="25.4"/>
-</segment>
 </net>
 <net name="+5V" class="0">
@@
 <label x="50.8" y="177.8" size="1.778" layer="95"/>
 </segment>
-<segment>
-<pinref part="LED1" gate="G$1" pin="A"/>
-<wire x1="43.18" y1="57.15" x2="43.18" y2="62.23" width="0.1524" layer="91"/>
-<label x="40.64" y="62.23" size="1.778" layer="95"/>
-</segment>
-<segment>
-<pinref part="LED2" gate="G$1" pin="A"/>
-<wire x1="68.58" y1="57.15" x2="68.58" y2="62.23" width="0.1524" layer="91"/>
-<label x="66.04" y="62.23" size="1.778" layer="95"/>
-</segment>
-<segment>
-<pinref part="LED3" gate="G$1" pin="A"/>
-<wire x1="93.98" y1="57.15" x2="93.98" y2="62.23" width="0.1524" layer="91"/>
-<label x="91.44" y="62.23" size="1.778" layer="95"/>
-</segment>
 </net>
 <net name="+12V" class="0">
@@
 </segment>
 </net>
-<net name="N$1" class="0">
-<segment>
-<pinref part="IC2" gate="A" pin="O"/>
-<wire x1="33.02" y1="54.61" x2="33.02" y2="39.37" width="0.1524" layer="91"/>
-<pinref part="U$1" gate="G$1" pin="B"/>
-<wire x1="33.02" y1="39.37" x2="38.1" y2="39.37" width="0.1524" layer="91"/>
-</segment>
-</net>
-<net name="N$2" class="0">
-<segment>
-<pinref part="IC2" gate="B" pin="O"/>
-<wire x1="58.42" y1="54.61" x2="58.42" y2="39.37" width="0.1524" layer="91"/>
-<pinref part="U$1" gate="G$2" pin="B"/>
-<wire x1="58.42" y1="39.37" x2="63.5" y2="39.37" width="0.1524" layer="91"/>
-</segment>
-</net>
-<net name="N$3" class="0">
-<segment>
-<pinref part="IC2" gate="C" pin="O"/>
-<wire x1="83.82" y1="54.61" x2="83.82" y2="39.37" width="0.1524" layer="91"/>
-<pinref part="U$2" gate="G$1" pin="B"/>
-<wire x1="83.82" y1="39.37" x2="88.9" y2="39.37" width="0.1524" layer="91"/>
-</segment>
-</net>
-<net name="N$5" class="0">
-<segment>
-<pinref part="U$1" gate="G$1" pin="C"/>
-<pinref part="LED1" gate="G$1" pin="C"/>
-<wire x1="43.18" y1="44.45" x2="43.18" y2="49.53" width="0.1524" layer="91"/>
-</segment>
-</net>
-<net name="N$8" class="0">
-<segment>
-<pinref part="U$1" gate="G$2" pin="C"/>
-<pinref part="LED2" gate="G$1" pin="C"/>
-<wire x1="68.58" y1="44.45" x2="68.58" y2="49.53" width="0.1524" layer="91"/>
-</segment>
-</net>
-<net name="N$9" class="0">
-<segment>
-<pinref part="U$2" gate="G$1" pin="C"/>
-<pinref part="LED3" gate="G$1" pin="C"/>
-<wire x1="93.98" y1="44.45" x2="93.98" y2="49.53" width="0.1524" layer="91"/>
-</segment>
-</net>
