File: Schematic/mainboard/T04_Main_Board.brd (EAGLE design)
At the start: 78.4 x 38.1 mm, 29 parts, among them IC1 7805DT, J1 AVR_SPI_PRG_6PTH, U1 ATMEGA328P_PDIP, X1 22-23-2021, X2 22-23-2071, X3 22-23-2081, Y1 16MHZ

Commit message: Mainboard Rev 1.3 Update
Parts:
- moved C1 1.27 mm to (64.8, 22.9)
- moved C3 1.27 mm to (31.8, 33.0)
- moved C4 1.27 mm to (27.9, 33.0)
- moved C5 1.27 mm to (20.3, 33.0)
- moved C6 1.27 mm to (24.1, 33.0)
- moved IC1 1.27 mm to (68.6, 14.0)
- moved TP12 1.27 mm to (72.4, 19.1)
- moved X1 1.27 mm to (71.1, 24.1)
Routing:
- net +5V: track 182.9 -> 179.1 mm
- net SCK: track 44.4 -> 41.9 mm
- net +12V: track 17.3 -> 18.0 mm
Other:
- board size 78.4 x 38.1 mm -> 75.9 x 38.1 mm
- board text added: "T04 Rev 1.3 November 9th, 2014 B. Driver N.Erickson D. Frister R.Wiseman"
- board text removed: "T04 Rev 1.0 B. Driver N.Erickson D. Frister R.Wiseman"

Commit message: Rev 1.4 Schematics/Layouts
Parts:
- removed JP1: (no value), SparkFun-Connectors:1X06-SMD
- added JP2: FTDI_BASICPTH, SparkFun-Connectors:FTDI_BASIC
- moved TP10 12.7 mm to (47.0, 15.2)
- moved TP11 12.7 mm to (49.5, 15.2)
- moved TP7 12.7 mm to (39.4, 15.2)
- moved TP8 12.7 mm to (41.9, 15.2)
- moved TP9 12.7 mm to (44.5, 15.2)
- moved TP6 11.4 mm to (36.8, 14.0)
- moved C8 1.27 mm to (7.62, 27.9)
Connections:
- net +5V: no longer JP1.4
- net BIT0: now also JP2.TXO; no longer JP1.2
- net BIT1: now also JP2.RXI; no longer JP1.3
- net CTS: now also JP2.CTS; no longer JP1.5
- net DTR: now also JP2.DTR; no longer JP1.1
- net GND: now also JP2.GND; no longer JP1.6
Routing:
- net +5V: track 179.1 -> 143.5 mm, vias 4 -> 2
- net BIT1: track 34.4 -> 43.2 mm
- net TRIG1: track 27.9 -> 22.9 mm
- net DTR: track 2.57 -> 6.35 mm
- net BIT0: track 35.9 -> 39.4 mm
- net ECHO3: track 27.9 -> 30.5 mm
- net TRIG3: track 17.8 -> 20.3 mm
- net TRIG2: track 17.8 -> 20.3 mm
- net ECHO2: track 17.8 -> 20.3 mm
- net ECHO1: track 17.8 -> 20.3 mm
- net RESET: track 92.7 -> 94.0 mm
- net +12V: track 18.0 -> 17.0 mm

Commit message: Final Schematic - Mainboard
Parts:
- removed Y1: 16MHZ, SparkFun-FreqCtrl:RESONATOR-SMD
- added C10, C9: 18p, rcl:C1206
- added Q1: 16MHz, special:QS
- C1, C2, C3, C4, C5, C6, C7, C8: device rcl:C025-024X044 -> rcl:C1206
- IC1: value 7805DT -> 7805TV; device linear:TO252 -> linear:TO220V
- R1: device rcl:M2309 -> rcl:R1206
- moved C6 48.8 mm to (62.2, 2.54), turned to 180 degrees
- moved C5 48.6 mm to (61.0, 6.35)
- moved C3 45.0 mm to (66.0, 3.81), turned to 270 degrees
- moved C4 44.5 mm to (63.5, 6.35)
- moved C2 42.3 mm to (30.5, 35.6), turned to 0 degrees
- moved C7 38.9 mm to (68.6, 8.89)
- moved IC1 4.02 mm to (67.3, 17.8), turned to 0 degrees
- moved U1 3.81 mm to (30.5, 27.9)
- moved TP6 1.27 mm to (36.8, 12.7)
- moved X2 1.27 mm to (24.1, 6.35)
- moved X3 1.27 mm to (45.7, 6.35)
- moved R1 1.27 mm to (58.4, 15.2)
Connections:
- removed net N$1: U1.9, Y1.1
- new net N$3: C9.2, Q1.1, U1.9
- net +5V: now also IC1.3; no longer IC1.2
- net GND: now also C10.1, C9.1, IC1.2; no longer IC1.3, Y1.2
- net N$2: now also C10.2, Q1.2; no longer Y1.3
Routing:
- net +5V: track 143.5 -> 173.6 mm, vias 2 -> 3
- net N$3: track 0.00 -> 11.3 mm
- net N$2: track 2.82 -> 10.8 mm
- net MUXENABLE: track 63.5 -> 71.1 mm
- net TRIG1: track 22.9 -> 29.7 mm
- net TRIG3: track 20.3 -> 26.7 mm
- net TRIG2: track 20.3 -> 26.7 mm
- net ECHO2: track 20.3 -> 26.7 mm
- net ECHO1: track 20.3 -> 26.7 mm
- net ECHO3: track 30.5 -> 36.8 mm
- net MISO: track 41.2 -> 45.0 mm
- net BIT0: track 39.4 -> 43.2 mm
- net BIT3: track 17.8 -> 21.6 mm
- net BIT2: track 17.8 -> 21.6 mm
- net SCK: track 41.9 -> 45.7 mm
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