File: Schematic/mainboard/T04_Main_Board.sch (EAGLE design)
At the start: 29 parts, among them IC1 7805DT, J1 AVR_SPI_PRG_6PTH, U1 ATMEGA328P_PDIP, X1 22-23-2021, X2 22-23-2071, X3 22-23-2081, Y1 16MHZ

Commit message: Rev 1.4 Schematics/Layouts
Parts:
- removed JP1: (no value), SparkFun-Connectors:ARDUINO_SERIAL_PROGRAMSMD
- added JP2: FTDI_BASICPTH, SparkFun-Connectors:FTDI_BASICPTH
Connections:
- net +5V: no longer JP1.VCC
- net BIT0: now also JP2.3; no longer JP1.RXI
- net BIT1: now also JP2.2; no longer JP1.TXO
- net CTS: now also JP2.5; no longer JP1.CTS
- net DTR: now also JP2.1; no longer JP1.DTR
- net GND: now also JP2.6; no longer JP1.GND
Changed lines of the file:
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@@
 <part name="GND7" library="supply1" deviceset="GND" device=""/>
 <part name="P+5" library="supply1" deviceset="+5V" device=""/>
-<part name="JP1" library="SparkFun-Connectors" deviceset="ARDUINO_SERIAL_PROGRAM" device="SMD"/>
 <part name="C8" library="rcl" deviceset="C-EU" device="025-024X044" value=".1u"/>
-<part name="P+3" library="supply1" deviceset="+5V" device=""/>
 <part name="GND9" library="supply1" deviceset="GND" device=""/>
 <part name="X2" library="con-molex" deviceset="22-23-2071" device=""/>
+<part name="JP2" library="SparkFun-Connectors" deviceset="FTDI_BASIC" device="PTH"/>
 </parts>
 <sheets>
@@
 <text x="289.56" y="147.32" size="1.778" layer="97">Connnector to sensors</text>
 <text x="274.32" y="109.22" size="1.778" layer="97">Connector to programmer</text>
-<wire x1="292.1" y1="213.36" x2="314.96" y2="213.36" width="0.1524" layer="97"/>
-<wire x1="314.96" y1="213.36" x2="314.96" y2="187.96" width="0.1524" layer="97"/>
-<wire x1="314.96" y1="187.96" x2="292.1" y2="187.96" width="0.1524" layer="97"/>
+<wire x1="292.1" y1="213.36" x2="317.5" y2="213.36" width="0.1524" layer="97"/>
+<wire x1="317.5" y1="213.36" x2="317.5" y2="187.96" width="0.1524" layer="97"/>
+<wire x1="317.5" y1="187.96" x2="292.1" y2="187.96" width="0.1524" layer="97"/>
 <wire x1="292.1" y1="187.96" x2="292.1" y2="213.36" width="0.1524" layer="97"/>
 <text x="292.1" y="214.63" size="1.778" layer="97">Serial Programmer</text>
@@
 <instance part="GND7" gate="1" x="180.34" y="149.86"/>
 <instance part="P+5" gate="1" x="177.8" y="162.56"/>
-<instance part="JP1" gate="G$1" x="304.8" y="198.12" rot="MR0"/>
 <instance part="C8" gate="G$1" x="162.56" y="177.8" rot="R180"/>
-<instance part="P+3" gate="1" x="271.78" y="208.28"/>
 <instance part="GND9" gate="1" x="284.48" y="203.2"/>
 <instance part="X2" gate="-1" x="304.8" y="172.72"/>
@@
 <instance part="X2" gate="-6" x="304.8" y="160.02"/>
 <instance part="X2" gate="-7" x="304.8" y="157.48"/>
+<instance part="JP2" gate="G$1" x="309.88" y="198.12" rot="MR0"/>
 </instances>
 <busses>
@@
 </segment>
 <segment>
-<pinref part="JP1" gate="G$1" pin="GND"/>
-<wire x1="299.72" y1="205.74" x2="289.56" y2="205.74" width="0.1524" layer="91"/>
+<wire x1="304.8" y1="205.74" x2="289.56" y2="205.74" width="0.1524" layer="91"/>
 <label x="294.64" y="205.74" size="1.778" layer="95"/>
 <wire x1="289.56" y1="205.74" x2="289.56" y2="210.82" width="0.1524" layer="91"/>
@@
 <wire x1="284.48" y1="210.82" x2="284.48" y2="205.74" width="0.1524" layer="91"/>
 <pinref part="GND9" gate="1" pin="GND"/>
+<pinref part="JP2" gate="G$1" pin="6"/>
 </segment>
 </net>
@@
 <junction x="185.42" y="160.02"/>
 </segment>
-<segment>
-<pinref part="JP1" gate="G$1" pin="VCC"/>
-<wire x1="299.72" y1="200.66" x2="271.78" y2="200.66" width="0.1524" layer="91"/>
-<label x="294.64" y="200.66" size="1.778" layer="95"/>
-<wire x1="271.78" y1="200.66" x2="271.78" y2="205.74" width="0.1524" layer="91"/>
-<pinref part="P+3" gate="1" pin="+5V"/>
-</segment>
 </net>
 <net name="+12V" class="0">
@@
 <wire x1="241.3" y1="142.24" x2="251.46" y2="142.24" width="0.1524" layer="91"/>
 <wire x1="251.46" y1="142.24" x2="251.46" y2="172.72" width="0.1524" layer="91"/>
-<wire x1="251.46" y1="172.72" x2="274.32" y2="172.72" width="0.1524" layer="91"/>
+<wire x1="251.46" y1="172.72" x2="269.24" y2="172.72" width="0.1524" layer="91"/>
 <label x="241.3" y="142.24" size="1.778" layer="95"/>
 <label x="294.64" y="172.72" size="1.778" layer="95"/>
 <pinref part="TP2" gate="G$1" pin="TP"/>
-<wire x1="274.32" y1="172.72" x2="276.86" y2="172.72" width="0.1524" layer="91"/>
+<wire x1="269.24" y1="172.72" x2="276.86" y2="172.72" width="0.1524" layer="91"/>
 <wire x1="276.86" y1="172.72" x2="302.26" y2="172.72" width="0.1524" layer="91"/>
 <junction x="276.86" y="172.72"/>
-<pinref part="JP1" gate="G$1" pin="RXI"/>
-<wire x1="274.32" y1="172.72" x2="274.32" y2="195.58" width="0.1524" layer="91"/>
-<wire x1="274.32" y1="195.58" x2="299.72" y2="195.58" width="0.1524" layer="91"/>
-<junction x="274.32" y="172.72"/>
-<label x="294.64" y="195.58" size="1.778" layer="95"/>
 <pinref part="X2" gate="-1" pin="S"/>
 <junction x="302.26" y="172.72"/>
+<wire x1="304.8" y1="198.12" x2="269.24" y2="198.12" width="0.1524" layer="91"/>
+<label x="294.64" y="198.12" size="1.778" layer="95"/>
+<wire x1="269.24" y1="198.12" x2="269.24" y2="172.72" width="0.1524" layer="91"/>
+<junction x="269.24" y="172.72"/>
+<pinref part="JP2" gate="G$1" pin="3"/>
 </segment>
 </net>
 <net name="BIT1" class="0">
 <segment>
-<pinref part="JP1" gate="G$1" pin="TXO"/>
 <wire x1="302.26" y1="170.18" x2="279.4" y2="170.18" width="0.1524" layer="91"/>
-<wire x1="279.4" y1="170.18" x2="271.78" y2="170.18" width="0.1524" layer="91"/>
-<wire x1="271.78" y1="170.18" x2="254" y2="170.18" width="0.1524" layer="91"/>
+<wire x1="279.4" y1="170.18" x2="274.32" y2="170.18" width="0.1524" layer="91"/>
+<wire x1="274.32" y1="170.18" x2="254" y2="170.18" width="0.1524" layer="91"/>
 <wire x1="254" y1="170.18" x2="254" y2="139.7" width="0.1524" layer="91"/>
 <pinref part="U1" gate="G$1" pin="PD1(TXD)"/>
@@
 <pinref part="TP3" gate="G$1" pin="TP"/>
 <junction x="279.4" y="170.18"/>
-<wire x1="299.72" y1="198.12" x2="271.78" y2="198.12" width="0.1524" layer="91"/>
-<wire x1="271.78" y1="198.12" x2="271.78" y2="170.18" width="0.1524" layer="91"/>
-<junction x="271.78" y="170.18"/>
-<label x="294.64" y="198.12" size="1.778" layer="95"/>
 <pinref part="X2" gate="-2" pin="S"/>
 <junction x="302.26" y="170.18"/>
+<wire x1="274.32" y1="195.58" x2="304.8" y2="195.58" width="0.1524" layer="91"/>
+<label x="294.64" y="195.58" size="1.778" layer="95"/>
+<wire x1="274.32" y1="195.58" x2="274.32" y2="170.18" width="0.1524" layer="91"/>
+<junction x="274.32" y="170.18"/>
+<pinref part="JP2" gate="G$1" pin="2"/>
 </segment>
 </net>
@@
 <net name="CTS" class="0">
 <segment>
-<pinref part="JP1" gate="G$1" pin="CTS"/>
-<wire x1="299.72" y1="203.2" x2="294.64" y2="203.2" width="0.1524" layer="91"/>
 <label x="294.64" y="203.2" size="1.778" layer="95"/>
+<pinref part="JP2" gate="G$1" pin="5"/>
+<wire x1="304.8" y1="203.2" x2="294.64" y2="203.2" width="0.1524" layer="91"/>
 </segment>
 </net>
@@
 </segment>
 <segment>
-<pinref part="JP1" gate="G$1" pin="DTR"/>
-<wire x1="299.72" y1="193.04" x2="294.64" y2="193.04" width="0.1524" layer="91"/>
 <label x="294.64" y="193.04" size="1.778" layer="95"/>
-</segment>
-</net>
+<pinref part="JP2" gate="G$1" pin="1"/>
+<wire x1="304.8" y1="193.04" x2="294.64" y2="193.04" width="0.1524" layer="91"/>
+</segment>
+</net>

Commit message: Final Schematic - Mainboard
Parts:
- removed Y1: 16MHZ, SparkFun-FreqCtrl:RESONATOR16MHZ
- added C10, C9: 18p, rcl:C-EUC1206
- added Q1: 16MHz, special:XTAL/S
- C1, C2, C3, C4, C5, C6, C7, C8: device rcl:C-EU025-024X044 -> rcl:C-EUC1206
- IC1: value 7805DT -> 7805TV; device linear:7805DT -> linear:7805TV
- R1: device rcl:R-US_M2309 -> rcl:R-US_R1206
Connections:
- removed net N$1: U1.PB6(XTAL1/TOSC1), Y1.1
- new net N$3: C9.2, Q1.1, U1.PB6(XTAL1/TOSC1)
- net GND: now also C10.1, C9.1; no longer Y1.2
- net N$2: now also C10.2, Q1.2; no longer Y1.3
